File: Dokumente/PCB_KiCad/Translator.sch (KiCad schematic (older format))
At the start: 17 parts, among them IC1 ATMEGA324A-P, P1 CONN_4X2, P2 CONN_4X2, P3 CONN_4X2, P4 CONN_4X2, P5 C64AC, U1 MAX232, U2 MAX232, X1 CRYSTAL

Commit message: Schaltplan und Platinenlayout aktualisiert
Connections:
- net at IC1.18 ((PCINT28/XCK1/OC1B)PD4), P5.A16 (16A): now also P5.C16 (16C)
- net at IC1.19 ((PCINT294/OC1A)PD5), P5.A17 (17A): now also P5.C17 (17C)
Changed lines of the file:
@@
-EESchema Schematic File Version 2  date 07.12.2011 20:17:46
+EESchema Schematic File Version 2  date 19.12.2011 18:43:26
 LIBS:power
 LIBS:device
@@
 Sheet 1 1
 Title "noname.sch"
-Date "7 dec 2011"
+Date "19 dec 2011"
 Rev ""
 Comp ""
@@
 $EndDescr
 Wire Wire Line
+	10200 4050 10200 3950
+Wire Wire Line
 	9600 5000 9600 3750
 Wire Wire Line
@@
 Wire Wire Line
 	9600 3750 10200 3750
+Wire Wire Line
+	10200 3750 10200 3850
 $Comp
 L CONN_4X2 P4
@@
 $EndComp
 $Comp
-L PWR_FLAG #FLG01
+L PWR_FLAG #FLG2
 U 1 1 4EDF8DDF
 P 9950 4450
-F 0 "#FLG01" H 9950 4545 30  0001 C CNN
+F 0 "#FLG2" H 9950 4545 30  0001 C CNN
 F 1 "PWR_FLAG" H 9950 4630 30  0000 C CNN
 	1    9950 4450
@@
 $EndComp
 $Comp
-L PWR_FLAG #FLG02
+L PWR_FLAG #FLG1
 U 1 1 4EDF8D2B
 P 9800 3350
-F 0 "#FLG02" H 9800 3445 30  0001 C CNN
+F 0 "#FLG1" H 9800 3445 30  0001 C CNN
 F 1 "PWR_FLAG" H 9800 3530 30  0000 C CNN
 	1    9800 3350
@@
 $EndComp
 $Comp
-L +5V #PWR03
+L +5V #PWR2
 U 1 1 4EDF8B1E
 P 1650 2600
-F 0 "#PWR03" H 1650 2690 20  0001 C CNN
+F 0 "#PWR2" H 1650 2690 20  0001 C CNN
 F 1 "+5V" H 1650 2690 30  0000 C CNN
 	1    1650 2600
@@
 $EndComp
 $Comp
-L GND #PWR04
+L GND #PWR10
 U 1 1 4EDF8969
 P 10050 4450
-F 0 "#PWR04" H 10050 4450 30  0001 C CNN
+F 0 "#PWR10" H 10050 4450 30  0001 C CNN
 F 1 "GND" H 10050 4380 30  0001 C CNN
 	1    10050 4450
@@
 $EndComp
 $Comp
-L +5V #PWR05
+L +5V #PWR9
 U 1 1 4EDF8943
 P 10000 3350
-F 0 "#PWR05" H 10000 3440 20  0001 C CNN
+F 0 "#PWR9" H 10000 3440 20  0001 C CNN
 F 1 "+5V" H 10000 3440 30  0000 C CNN
 	1    10000 3350
@@
 $EndComp
 $Comp
-L +5V #PWR06
+L +5V #PWR1
 U 1 1 4EDF87F6
 P 1650 1400
-F 0 "#PWR06" H 1650 1490 20  0001 C CNN
+F 0 "#PWR1" H 1650 1490 20  0001 C CNN
 F 1 "+5V" H 1650 1490 30  0000 C CNN
 	1    1650 1400
@@
 $EndComp
 $Comp
-L +5V #PWR07
+L +5V #PWR7
 U 1 1 4EDF838E
 P 7300 3300
-F 0 "#PWR07" H 7300 3390 20  0001 C CNN
+F 0 "#PWR7" H 7300 3390 20  0001 C CNN
 F 1 "+5V" H 7300 3390 30  0000 C CNN
 	1    7300 3300
@@
 $EndComp
 $Comp
-L +5V #PWR08
+L +5V #PWR5
 U 1 1 4EDF8376
 P 7300 1400
-F 0 "#PWR08" H 7300 1490 20  0001 C CNN
+F 0 "#PWR5" H 7300 1490 20  0001 C CNN
 F 1 "+5V" H 7300 1490 30  0000 C CNN
 	1    7300 1400
@@
 $EndComp
 $Comp
-L GND #PWR09
+L GND #PWR6
 U 1 1 4EDF836A
 P 7300 2000
-F 0 "#PWR09" H 7300 2000 30  0001 C CNN
+F 0 "#PWR6" H 7300 2000 30  0001 C CNN
 F 1 "GND" H 7300 1930 30  0001 C CNN
 	1    7300 2000
@@
 $EndComp
 $Comp
-L GND #PWR010
+L GND #PWR8
 U 1 1 4EDF8165
 P 7300 3900
-F 0 "#PWR010" H 7300 3900 30  0001 C CNN
+F 0 "#PWR8" H 7300 3900 30  0001 C CNN
 F 1 "GND" H 7300 3830 30  0001 C CNN
 	1    7300 3900
@@
 $EndComp
 $Comp
-L GND #PWR011
+L GND #PWR4
 U 1 1 4EDF8148
 P 2450 5200
-F 0 "#PWR011" H 2450 5200 30  0001 C CNN
+F 0 "#PWR4" H 2450 5200 30  0001 C CNN
 F 1 "GND" H 2450 5130 30  0001 C CNN
 	1    2450 5200
@@
 $EndComp
 $Comp
-L +5V #PWR012
+L +5V #PWR3
 U 1 1 4EDF8128
 P 2450 1100
-F 0 "#PWR012" H 2450 1190 20  0001 C CNN
+F 0 "#PWR3" H 2450 1190 20  0001 C CNN
 F 1 "+5V" H 2450 1190 30  0000 C CNN
 	1    2450 1100

Commit message: commit?
Parts:
- removed P1, P2, P3, P4: CONN_4X2, symbol CONN_4X2
- removed P5: C64AC, symbol C64AC
- added P1: CONN_2, symbol CONN_2
- added P2: SWITCH, symbol CONN_5X2
- added P3: LED, symbol CONN_5X2
- added P4: LCD, symbol CONN_5X2
- added P5: RS-232 RF, symbol CONN_5X2
- added P6: RS-232 ST, symbol CONN_5X2
- added P7: C64AC, symbol C64AC
- added R1, R10, R11, R12, R13, R14, R15, R2, R3, R4, R5, R6, R7, R8, R9: 150R, symbol R
- added RV1: POT, symbol POT
- U1: value MAX232 -> MAX232 RF
- U2: value MAX232 -> MAX232 ST
Connections:
- net +5V: now also P1.1 (P1), P3.10, P3.2, P3.4, P3.6, P3.8, P4.9, P7.A14 (14A), P7.C14 (14C), R11.2, R12.2, R13.2, R14.2, R15.2, RV1.3; no longer IC1.9 (~RESET)
- net GND: now also U1.10 (T2IN), U2.10 (T2IN), P2.10, P2.2, P2.4, P2.6, P2.8, P4.10, P5.9, P6.9, P7.A19 (19A), P7.C19 (19C), RV1.1
- net at IC1.18 ((PCINT28/XCK1/OC1B)PD4): now also P7.A17 (17A), P7.C17 (17C)
- net at IC1.19 ((PCINT294/OC1A)PD5): now also P7.A16 (16A), P7.C16 (16C)
- net at IC1.1 ((PCINT8/T0/XCK)PB0): now also R6.1
- net at IC1.2 ((PCINT9/CLKO/T1)PB1): now also R7.1
- net at IC1.22 ((PCINT16/SCL)PC0): now also P4.1
- net at IC1.23 ((PCINT17/SDA)PC1): now also P4.2
- net at IC1.24 ((PCINT18/TCK)PC2): now also P4.3
- net at IC1.25 ((PCINT19/TMS)PC3): now also P4.4
- net at IC1.26 ((PCINT20/TDO)PC4): now also P4.5
- net at IC1.27 ((PCINT21/TDI)PC5): now also P4.6
- net at IC1.28 ((PCINT22/TOSC1)PC6): now also P4.7
- net at IC1.3 ((PCINT10/AIN0/INT2)PB2): now also R8.1
- net at IC1.36 ((PCINT4/ADC4)PA4): now also R5.1
- net at IC1.37 ((PCINT3/ADC3)PA3): now also R4.1
- net at IC1.38 ((PCINT2/ADC2)PA2): now also R3.1
- net at IC1.39 ((PCINT1/ADC1)PA1): now also R2.1
- net at IC1.4 ((PCINT11/AIN1/OC0)PB3): now also R9.1
- net at IC1.40 ((PCINT0/ADC0)PA0): now also R1.1
- net at IC1.5 ((PCINT12/OC0B/~SS~)PB4): now also R10.1
- net at U1.9 (R2OUT): no longer U1.10 (T2IN)
- net at U1.13 (R1IN): now also P5.5
- net at U1.14 (T1OUT): now also P5.3
- net at U1.7 (T2OUT): now also P5.1, P5.2
- net at U2.9 (R2OUT): no longer U2.10 (T2IN)
- net at U2.13 (R1IN): now also P6.5
- net at U2.14 (T1OUT): now also P6.3
- net at U2.7 (T2OUT): now also P6.1, P6.2
- new net: IC1.9 (~RESET), P1.2 (PM)
- new net: P2.1, R1.2, R11.1
- new net: P2.3, R12.1, R2.2
- new net: P2.5, R13.1, R3.2
- new net: P2.7, R14.1, R4.2
- new net: P2.9, R15.1, R5.2
- new net: P3.1, R6.2
- new net: P3.3, R7.2
- new net: P3.5, R8.2
- new net: P3.7, R9.2
- new net: P3.9, R10.2
- new net: P4.8, RV1.2
- new net: P6.4, P6.6
- new net: P5.4, P5.6
- no-connect marks 0 -> 75
Other:
- moved on the sheet: C1, C2, C3, C4, C5, C6, C7, C8, U1, U2
